File: th-lora/th-lora.sch (EAGLE design)
At the start: 23 parts, among them J2 AVR_SPI_PRG_6NS, X1 SMA-142-0701-801/806, X2 UBLOX_MAX, X3 RFM98

Commit message: finishing off
Parts:
- removed C13, C14: (no value), rcl:C-EU050-025X075
- removed JP3: FTDI_BASICPTH, SparkFun-Connectors:FTDI_BASICPTH
- removed LED3: (no value), dtb:LED3MM
- removed R8: (no value), rcl:R-EU_0204/7
- removed S1: SWITCH-MOMENTARY-2SMD, Mine:SWITCH-MOMENTARY-2SMD
- removed U$2: TINY2313-*P*, avr-7:TINY2313-*P*
- removed U$5: JTI_ANTENNA-1575AT43A40, Ava:JTI_ANTENNA-1575AT43A40
- added C2, C3: 27p, rcl:C-EU050-025X075
- added C4: 100n, rcl:C-EU050-025X075
- added C6: 10u, rcl:CPOL-EUE2.5-5
- added IC1: TINY2313-*P*, avr-7:TINY2313-*P*
- added IC2: MCP1700, dtb:MCP1700
- added JP2: M023.5MM, SparkFun-Connectors:M023.5MM
- added LED1: (no value), dtb:LED3MM
- added R1: 330, rcl:R-EU_0204/7
- added R2: 10k, rcl:R-EU_0204/7
- C1, C5, C8: value (none) -> 1u
- C7: value (none) -> 100n
- J1: value (none) -> AVR_SPI_PRG_6NS; device dtb:JST_2MM_MALE -> SparkFun-Connectors:AVR_SPI_PRG_6NS
- J2: value AVR_SPI_PRG_6NS -> (none); device SparkFun-Connectors:AVR_SPI_PRG_6NS -> dtb:JST_2MM_MALE
- JP1: value M023.5MM -> FTDI_BASICPTH; device SparkFun-Connectors:M023.5MM -> SparkFun-Connectors:FTDI_BASICPTH
- R3: value (none) -> 10k
- U$3: value MCP1700 -> JTI_ANTENNA-1575AT43A40; device dtb:MCP1700 -> Ava:JTI_ANTENNA-1575AT43A40
- X2: value UBLOX_MAX -> RFM98; device Ava:UBLOX_MAX -> Mine:RFM98
- X3: value RFM98 -> UBLOX_MAX; device Mine:RFM98 -> Ava:UBLOX_MAX
- renumbered C10 to C7, C11 to C5, C12 to C8, L2 to L1
Connections:
- removed net N$15: U$2.(AIN0)PB0
- removed net N$5: S1.2
- removed net N$8: S1.1
- removed net SCLK: X3.SCK
- new net N$13: JP1.3, R3.2, X3.3_RXD1
- new net R_RST: IC1.(OC1B)PB4, X2.RST
- net +3V3: now also C4.1, C6.+, IC1.VCC, IC2.OUT, J1.2, JP1.4, X2.3.3V, X3.6_V_BCKP, X3.7_VCC_IO, X3.8_VCC; no longer J2.2, JP3.4, U$2.VCC, U$3.OUT, X2.6_V_BCKP, X2.7_VCC_IO, X2.8_VCC, X3.3.3V
- net GND: now also C2.1, C3.1, C4.2, C6.-, IC1.GND, IC2.GND, J1.6, J2.-, JP1.6, JP2.2, R1.1, X2.GND, X3.10_GND, X3.12_GND, X3.1_GND; no longer C13.1, C14.1, J1.-, J2.6, JP1.1, JP3.6, R8.1, U$2.GND, U$3.GND, X2.10_GND, X2.12_GND, X2.1_GND, X3.GND
- net MISO: now also IC1.(MISO)PB6, J1.1, R2.2; no longer J2.1, U$2.(MISO)PB6, X3.MISO
- net MOSI: now also IC1.(MOSI)PB5, J1.4, X2.MOSI; no longer J2.4, U$2.(MOSI)PB5, X3.MOSI
- net N$1: now also X3.11_RF_IN; no longer X2.11_RF_IN
- net N$11: now also IC2.IN, J2.+, JP2.1; no longer J1.+, JP1.2, U$3.IN
- net N$12: now also IC1.(INT0)PD2, LED1.A; no longer LED3.A, U$2.(T0)PD4
- net N$14: now also R2.1, X2.MISO; no longer R3.2, X2.2_TXD1
- net N$2: now also X2.ANT; no longer X3.ANT
- net N$3: now also LED1.C, R1.2; no longer LED3.C, R8.2
- net N$4: now also U$3.FEED; no longer U$5.FEED
- net N$6: now also C2.2, IC1.PA1(XTAL2); no longer C13.2, U$2.PA1(XTAL2)
- net N$7: now also C3.2, IC1.PA0(XTAL1); no longer C14.2, U$2.PA0(XTAL1)
- net NSS: now also IC1.(INT1)PD3, X2.NSS; no longer X3.NSS
- net RST: now also IC1.PA2(/RESET), J1.5; no longer J2.5, U$2.PA2(/RESET)
- net SCK: now also IC1.(UCSK)PB7, J1.3, X2.SCK; no longer J2.3, U$2.(UCSK)PB7
- net UART_RX: now also IC1.(RXD)PD0, JP1.2, X3.2_TXD1; no longer JP3.3, R3.1, U$2.(RXD)PD0
- net UART_TX: now also IC1.(TXD)PD1, R3.1; no longer JP3.2, U$2.(TXD)PD1, X2.3_RXD1
Other:
- moved on the sheet: C1, Q1, R3
