File: th-lora/th-lora.brd (EAGLE design)
At the start: 29.1 x 72.9 mm, 24 parts, among them J2 AVR_SPI_PRG_6NS, X1 SMA-142-0701-801/806, X2 UBLOX_MAX, X3 RFM98

Commit message: finishing off
Parts:
- removed C11, C14: (no value), rcl:C050-025X075
- removed JP3: FTDI_BASICPTH, SparkFun-Connectors:FTDI_BASIC
- removed L2: (no value), SparkFun-Passives:0603
- removed S1: SWITCH-MOMENTARY-2SMD, Mine:TACTILE_SWITCH_SMD
- removed U$5: JTI_ANTENNA-1575AT43A40, Ava:JTI_ANTENNA-1575AT43A40
- added C3: 27p, rcl:C050-025X075
- added C4: 100n, rcl:C050-025X075
- added C5: 1u, rcl:C050-025X075
- added C6: 10u, rcl:E2,5-5
- added IC2: MCP1700, dtb:TO92-INLINE
- added JP2: M023.5MM, SparkFun-Connectors:SCREWTERMINAL-3.5MM-2
- added L1: (no value), SparkFun-Passives:0603
- added R2: 10k, rcl:0204/7
- C1, C8: value (none) -> 1u
- C2: value (none) -> 27p
- C7: value (none) -> 100n
- J1: value (none) -> AVR_SPI_PRG_6NS; device dtb:JST-2-SMD -> SparkFun-Connectors:2X3-NS
- J2: value AVR_SPI_PRG_6NS -> (none); device SparkFun-Connectors:2X3-NS -> dtb:JST-2-SMD
- JP1: value M023.5MM -> FTDI_BASICPTH; device SparkFun-Connectors:SCREWTERMINAL-3.5MM-2 -> SparkFun-Connectors:FTDI_BASIC
- R1: value (none) -> 330
- R3: value (none) -> 10k
- U$3: value MCP1700 -> JTI_ANTENNA-1575AT43A40; device dtb:TO92-INLINE -> Ava:JTI_ANTENNA-1575AT43A40
- X2: value UBLOX_MAX -> RFM98; device Ava:UBLOX_MAX -> Mine:RFM97
- X3: value RFM98 -> UBLOX_MAX; device Mine:RFM97 -> Ava:UBLOX_MAX
- moved J2 53.4 mm to (26.0, 53.3), turned to 270 degrees
- moved J1 53.2 mm to (3.68, 5.08), turned to 90 degrees
- moved C1 37.5 mm to (24.9, 5.84), turned to 0 degrees
- moved X2 34.5 mm to (27.9, 24.8)
- moved X3 34.5 mm to (7.24, 52.3)
- moved JP1 28.0 mm to (2.16, 26.0), turned to 270 degrees
- moved U$3 20.6 mm to (10.5, 64.8)
- moved R3 2.41 mm to (6.22, 41.5)
- turned LED1 to 180 degrees
- renumbered C10 to C7, C12 to C8, C13 to C2, LED3 to LED1, R8 to R1, U$1 to U$4, U$2 to IC1
Connections:
- removed net N$15: IC1.12
- removed net N$5: S1.3
- removed net N$8: S1.1
- removed net SCLK: X3.4
- new net N$13: JP1.TXO, R3.2, X3.3_RXD1
- new net R_RST: IC1.16, X2.6
- net +3V3: now also C4.1, C5.1, C6.+, IC2.VOUT, J1.2, JP1.VCC, X2.13, X3.6_V_BCKP, X3.7_VCC_IO, X3.8_VCC; no longer C11.1, J2.2, JP3.VCC, U$3.VOUT, X2.6_V_BCKP, X2.7_VCC_IO, X2.8_VCC, X3.13
- net 9_V_RESET: now also X3.9_V_RESET; no longer X2.9_V_RESET
- net GND: now also C3.1, C4.2, C5.2, C6.-, IC2.GND, J1.6, J2.1, JP1.GND, JP2.2, L1.2, X2.1, X2.10, X2.8, X3.10_GND, X3.12_GND, X3.1_GND; no longer C11.2, C14.1, J1.1, J2.6, JP1.1, JP3.GND, L2.2, U$3.GND, X2.10_GND, X2.12_GND, X2.1_GND, X3.1, X3.10, X3.8
- net MISO: now also J1.1, R2.2; no longer J2.1, X3.2
- net MOSI: now also J1.4, X2.3; no longer J2.4, X3.3
- net N$1: now also X3.11_RF_IN; no longer X2.11_RF_IN
- net N$11: now also IC2.VIN, J2.2, JP2.1; no longer J1.2, JP1.2, U$3.VIN
- net N$12: now also IC1.6; no longer IC1.8
- net N$14: now also R2.1, X2.2; no longer R3.2, X2.2_TXD1
- net N$2: now also X2.9; no longer X3.9
- net N$4: now also L1.1, U$3.FEED; no longer L2.1, U$5.FEED
- net N$7: now also C3.2; no longer C14.2
- net NSS: now also IC1.7, X2.5; no longer X3.5
- net RST: now also J1.5; no longer J2.5
- net SCK: now also J1.3, X2.4; no longer J2.3
- net UART_RX: now also JP1.RXI, X3.2_TXD1; no longer JP3.TXO, R3.1
- net UART_TX: now also R3.1; no longer JP3.RXI, X2.3_RXD1
Routing:
- net GND: track 197.2 -> 127.8 mm, vias 4 -> 103
- net N$13: track 0.00 -> 39.2 mm, vias 0 -> 4
- net +3V3: track 110.3 -> 145.6 mm, vias 4 -> 2
- net UART_TX: track 38.6 -> 12.2 mm, vias 1 -> 0
- net SCK: track 36.4 -> 61.6 mm, vias 2 -> 4
- net R_RST: track 0.00 -> 22.2 mm, vias 0 -> 2
- net MOSI: track 69.9 -> 60.3 mm, vias 2 -> 0
- net MISO: track 65.7 -> 57.0 mm, vias 0 -> 1
- net NSS: track 0.00 -> 6.80 mm
- net N$3: track 7.51 -> 4.97 mm
- net N$12: track 23.0 -> 20.9 mm, vias 2 -> 0
- net RST: track 23.9 -> 24.2 mm, vias 1 -> 0
- added copper zone on layer 1, net GND
- added copper zone on layer 16, net GND
Other:
- board size 29.1 x 72.9 mm -> 29.1 x 69.1 mm
- board text added: "+"
- board text added: "-"
- board text added: "0V"
- board text added: "MI"
- board text added: "MO"
- board text added: "Max 6V"
- board text added: "SK"
- board text added: "V+"
- board text added: "VCC"

Commit message: adding copyright notice
Other:
- board text added: "©"
Changed lines of the file:
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@@
 <text x="27.178" y="41.656" size="1.4224" layer="22" font="vector" ratio="14" rot="MR0">+</text>
 <text x="26.162" y="45.466" size="1.4224" layer="22" font="vector" ratio="14" rot="MR90">-</text>
+<text x="25.654" y="10.668" size="1.27" layer="22" rot="MR0">©</text>
 </plain>
 <attributes>
