File: combined.brd (EAGLE design)
At the start: 73.4 x 45.5 mm, 64 parts, among them IC1 STM32F0, IC2 MCP1700TT, IC3 MCP73831, IC4 MCP1700TT, J1 SWD_SHROUD_SMD, Q1 BSS84, Q2 BSS84, SW1 ROTARTY_ENCODER, U1 NHD-C0216CIZ-FSW, U2 RFM98, U3 RN4020, X1 BU-SMA-V, X2 CRYSTAL-GROUNDED

Commit message: panelized
Parts:
- added C18, C19, C27, C28: 10u, rcl:C0805
- added C20, C24, C29, C33: 100n, rcl:C0603
- added C21, C23, C26, C30, C32, C35: 1u, rcl:C0603
- added C22, C31: 4u7, rcl:C0603
- added C25, C34, C36: (no value), rcl:C0603
- added C37, C42: 100n, rcl:C050-025X075
- added C38, C39, C43: 1u, rcl:C050-025X075
- added C40, C41: 27p, rcl:C050-025X075
- added C44: 10u, rcl:E2,5-5
- added IC10: MCP1700, dtb:TO92-INLINE
- added IC5, IC7: STM32F030F4, dtb:TSSOP20
- added IC6, IC8: ADP1607, Mine:LFCSP6
- added IC9: TINY2313-*P*, avr-7:DIL20
- added J3, J4: SWD_PTH_SHROUD, dtb:SWD_PTH_SHROUD
- added J5: AVR_SPI_PRG_6NS, SparkFun-Connectors:2X3-NS
- added J6: (no value), dtb:JST-2-SMD
- added JP3: M05X2SHD, SparkFun-Connectors:2X5-SHROUDED
- added JP4: M023.5MM, SparkFun-Connectors:SCREWTERMINAL-3.5MM-2
- added JP5: FTDI_BASICPTH, SparkFun-Connectors:FTDI_BASIC
- added L2, L5: 2u2, SparkFun-Passives:0805
- added L3, L6, L8: (no value), SparkFun-Passives:0603
- added L4, L7: (no value), SparkFun-Passives:1210
- added LED10: (no value), dtb:LED3MM
- added LED8, LED9: (no value), SparkFun-LED:LED-0603
- added Q3: (no value), crystal:HC49/S
- added R11, R2: 220k, rcl:R0603
- added R12, R8: 10k, rcl:R0603
- added R14: 330, rcl:0204/7
- added R15, R18: 10k, rcl:0204/7
- added R3, R9: 360k, rcl:R0603
- added R6, R7: 330, rcl:R0603
- added S4: SWITCH-MOMENTARY-2SMD, Mine:TACTILE_SWITCH_SMD
- added TP1, TP2, TP3, TP4, TP5, TP6: PTR1B1,27, testpad:B1,27
- added U$10, U$3, U$8: (no value), Mine:SUSF-XSM
- added U$4, U$5, U$9: JTI_ANTENNA-1575AT43A40, Ava:JTI_ANTENNA-1575AT43A40
- added U$6, U$7: KEYSTONE-53, Mine:KEYSTONE53
- added X10, X4, X7: SMA-142-0701-801/806, con-coax1:J502-ND-142-0701-801/806
- added X11, X5, X8: RFM98, Mine:RFM97
- added X3, X6, X9: UBLOX_MAX, Ava:UBLOX_MAX
- moved D1 0.90 mm to (65.4, 29.2)
- moved JP1 0.90 mm to (71.2, 23.5)
- moved L1 0.90 mm to (65.7, 26.0)
- moved U$1 0.90 mm to (71.1, 32.1)
- moved S2 0.90 mm to (42.5, 8.26)
- moved H4 0.90 mm to (69.2, 4.45)
- moved J1 0.90 mm to (70.1, 13.8)
- moved LED4 0.90 mm to (42.5, 14.6)
- moved R4 0.90 mm to (38.5, 15.6)
- moved SW1 0.90 mm to (55.9, 10.8)
- moved C4 0.90 mm to (30.4, 20.6)
- moved C12 0.90 mm to (55.9, 30.2)
- moved C14 0.90 mm to (47.6, 41.1)
- moved C15 0.90 mm to (26.2, 41.1)
- moved C16 0.90 mm to (50.5, 43.3)
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Connections:
- new net +3V1: C18.1, C20.1, C21.1, C22.1, C23.1, C24.1, IC5.16, IC5.5, IC6.6, J3.1, JP3.1, LED9.A, R3.2, X3.6_V_BCKP, X3.7_VCC_IO, X3.8_VCC, X5.13
- new net +3V2: C27.1, C29.1, C30.1, C31.1, C32.1, C33.1, IC7.16, IC7.5, IC8.6, J4.1, R9.2, X6.6_V_BCKP, X6.7_VCC_IO, X6.8_VCC, X8.13
- new net +3V4: C37.1, C38.1, C42.1, C43.1, C44.+, IC10.VOUT, IC9.20, J5.2, JP5.VCC, X11.13, X9.6_V_BCKP, X9.7_VCC_IO, X9.8_VCC
- new net 9_V_RESET: X3.9_V_RESET
- new net 9_V_RESET1: X6.9_V_RESET
- new net 9_V_RESET2: X9.9_V_RESET
- new net CLK: IC7.2, X8.7
- new net GND2: C27.2, C28.2, C29.2, C30.2, C31.2, C32.2, C33.2, C35.2, IC7.1, IC7.15, IC8.4, IC8.EP, J4.3, J4.5, J4.9, L6.2, R11.1, TP6.TP, U$7.N1, U$7.N2, X6.10_GND, X6.12_GND, X6.1_GND, X7.G@1, X7.G@2, X7.G@3, X7.G@4, X8.1, X8.10, X8.8
- new net GND3: C18.2, C19.2, C20.2, C21.2, C22.2, C23.2, C24.2, C26.2, C37.2, C38.2, C39.2, C40.1, C41.1, C42.2, C43.2, C44.-, IC10.GND, IC5.1, IC5.15, IC6.4, IC6.EP, IC9.10, J3.3, J3.5, J3.9, J5.6, J6.1, JP3.2, JP4.2, JP5.GND, L3.2, L8.2, LED8.C, R14.1, R2.1, S4.1, TP1.TP, U$6.N1, U$6.N2, X10.G@1, X10.G@2, X10.G@3, X10.G@4, X11.1, X11.10, X11.8, X3.10_GND, X3.12_GND, X3.1_GND, X4.G@1, X4.G@2, X4.G@3, X4.G@4, X5.1, X5.10, X5.8, X9.10_GND, X9.12_GND, X9.1_GND
- new net GPIO1: IC5.3, JP3.8
- new net GPIO2: IC5.2, JP3.9, X5.7
- new net GPIO3: IC5.6, JP3.10
- new net GPIO4: IC7.3
- new net GPIO5: IC7.6
- new net MISO1: IC5.12, JP3.7, X5.2
- new net MISO2: IC7.12, X8.2
- new net MISO3: IC9.18, J5.1, R18.2
- new net MOSI1: IC5.13, JP3.6, X5.3
- new net MOSI2: IC7.13, X8.3
- new net MOSI3: IC9.17, J5.4, X11.3
- new net N$19: X4.1, X5.9
- new net N$20: IC6.5, L2.2, L4.2
- new net N$21: IC6.3, R2.2, R3.1
- new net N$22: LED9.C, R7.2
- new net N$24: IC5.7, R8.2
- new net N$25: C25.2, X3.11_RF_IN
- new net N$26: C25.1, L3.1, U$5.FEED
- new net N$36: IC5.14, R6.2, R7.1
- new net N$37: LED8.A, R6.1, S4.3
- new net N$38: X5.6
- new net N$39: X7.1, X8.9
- new net N$40: IC8.5, L5.2, L7.2
- new net N$41: IC8.3, R11.2, R9.1
- new net N$42: IC7.7, R12.2
- new net N$43: C34.2, X6.11_RF_IN
- new net N$44: C34.1, L6.1, U$4.FEED
- new net N$45: X10.1, X11.9
- new net N$46: C36.2, X9.11_RF_IN
- new net N$47: C36.1, L8.1, U$9.FEED
- new net N$48: C39.1, IC10.VIN, J6.2, JP4.1
- new net N$49: C40.2, IC9.4, Q3.2
- new net N$50: C41.2, IC9.5, Q3.1
- new net N$51: LED10.K, R14.2
- new net N$52: IC9.6, LED10.A
- new net N$53: JP5.TXO, R15.2, X9.3_RXD1
- new net N$54: R18.1, X11.2
- new net NSS1: IC5.10, X5.5
- new net NSS2: IC7.10, X8.5
- new net NSS3: IC9.7, X11.5
- new net RST1: IC5.4, J3.10
- new net RST2: IC7.4, J4.10
- new net RST3: IC9.1, J5.5
- new net R_RST: IC9.16, X11.6
- new net SCK: IC9.19, J5.3, X11.4
- new net SCL1: IC5.17, JP3.3
- new net SCL2: IC7.17
- new net SCLK1: IC5.11, JP3.5, X5.4
- new net SCLK2: IC7.11, X8.4
- new net SDA1: IC5.18, JP3.4
- new net SDA2: IC7.18
- new net SWCLK1: IC5.20, J3.4
- new net SWCLK2: IC7.20, J4.4
- new net SWDAT1: IC5.19, J3.2
- new net SWDAT2: IC7.19, J4.2
- new net UART_RX: IC5.9, TP2.TP, X3.2_TXD1
- new net UART_RX1: IC7.9, TP4.TP, X6.2_TXD1
- new net UART_RX2: IC9.2, JP5.RXI, X9.2_TXD1
- new net UART_TX: IC5.8, TP3.TP, X3.3_RXD1
- new net UART_TX1: IC7.8, TP5.TP, X6.3_RXD1
- new net UART_TX2: IC9.3, R15.1
- new net VBAT: C19.1, C26.1, IC6.1, IC6.2, L2.1, L4.1, R8.1, U$6.P1, U$6.P2
- new net VBAT1: C28.1, C35.1, IC8.1, IC8.2, L5.1, L7.1, R12.1, U$7.P1, U$7.P2
Routing:
- net GND3: track 0.00 -> 175.0 mm, vias 0 -> 209
- net +3V4: track 0.00 -> 145.6 mm, vias 0 -> 2
- net +3V1: track 0.00 -> 144.8 mm, vias 0 -> 7
- net +3V2: track 0.00 -> 111.8 mm, vias 0 -> 6
- net VBAT: track 0.00 -> 72.4 mm, vias 0 -> 3
- net VBAT1: track 0.00 -> 62.2 mm, vias 0 -> 2
- net SCK: track 0.00 -> 61.6 mm, vias 0 -> 4
- net MOSI3: track 0.00 -> 60.3 mm
- net GND2: track 0.00 -> 59.3 mm, vias 0 -> 127
- net MISO3: track 0.00 -> 57.0 mm, vias 0 -> 1
- net N$53: track 0.00 -> 39.2 mm, vias 0 -> 4
- net N$36: track 0.00 -> 36.7 mm, vias 0 -> 3
- net SCLK1: track 0.00 -> 35.9 mm, vias 0 -> 1
- net RST1: track 0.00 -> 35.3 mm
- net MISO1: track 0.00 -> 31.8 mm, vias 0 -> 1
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- added copper zone on layer 1, net GND2
- added copper zone on layer 16, net GND2
- added copper zone on layer 1, net GND3
- added copper zone on layer 16, net GND3
Other:
- board size 73.4 x 45.5 mm -> 99.4 x 99.4 mm
- board text added: "+"
- board text added: "-"
- board text added: "0V"
- board text added: "C1"
- board text added: "C10"
- board text added: "C11"
- board text added: "C12"
- board text added: "C13"
- board text added: "C14"
- board text added: "C15"
- board text added: "C16"
- board text added: "C17"
- board text added: "C2"
- board text added: "C3"
- board text added: "C4"
- board text added: "C5"
- board text added: "C6"
- board text added: "C7"
- board text added: "C8"
- board text added: "C9"
- board text added: "D1"
- board text added: "GND"
- board text added: "IC1"
- board text added: "IC2"
- board text added: "IC3"
- board text added: "IC4"
- board text added: "J2"
- board text added: "L1"
- board text added: "L2"
- board text added: "MI"
- board text added: "MO"
- board text added: "Max 6V"
- board text added: "Phil Crump"
- board text added: "Q1"
- board text added: "Q2"
- board text added: "R"
- board text added: "R1"
- board text added: "R10"
- board text added: "R13"
- board text added: "R16"
- board text added: "R17"
- board text added: "R2"
- board text added: "R3"
- board text added: "R4"
- board text added: "R5"
- board text added: "RN1"
- board text added: "RN2"
- board text added: "RN3"
- board text added: "RX"
- board text added: "S1"
- board text added: "SK"
- board text added: "T"
- board text added: "TX"
- board text added: "V+"
- board text added: "VCC"
- board text added: "X1"
- board text added: "X2"

Commit message: prodding
Routing:
- net VBAT: track 72.4 -> 74.2 mm
- net GND: track 203.6 -> 204.9 mm, vias 144 -> 145
- net +3V1: track 144.8 -> 143.9 mm
Other:
- board text removed: "X1"

Commit message: sent off
Parts:
- moved U$10 48.8 mm to (8.64, 91.9)
Routing:
- net GND3: track 174.8 -> 175.1 mm, vias 209 -> 211
