File: basestation-board/basestation.brd (EAGLE design)
At the start: 73.4 x 45.5 mm, 64 parts, among them IC1 STM32F0, IC2 MCP1700TT, IC3 MCP73831, IC4 MCP1700TT, J1 SWD_SHROUD_SMD, Q1 BSS84, Q2 BSS84, SW1 ROTARTY_ENCODER, U1 NHD-C0216CIZ-FSW, U2 RFM98, U3 RN4020, X1 BU-SMA-V, X2 CRYSTAL-GROUNDED

Commit message: adding part values
Parts:
- C1, C13, C15, C3, C4, C9: value (none) -> 1u
- C10, C6: value (none) -> 27p
- C12, C5: value (none) -> 100n
- C2: value (none) -> 4u7
- Q1: value BSS84 -> NX2301
- R1: value (none) -> 10k
- R10, R17: value (none) -> 470
- R16: value (none) -> 4k7

Commit message: adding copyright notice
Parts:
- C1, C13, C15, C3, C4, C9: value 1u -> (none)
- C10, C6: value 27p -> (none)
- C12, C5: value 100n -> (none)
- C2: value 4u7 -> (none)
- Q1: value NX2301 -> BSS84
- R1: value 10k -> (none)
- R10, R17: value 470 -> (none)
- R16: value 4k7 -> (none)
Other:
- board text added: "©"
