File: basestation-board/basestation.sch (EAGLE design)
At the start: 70 parts, among them IC1 STM32F0, IC2 MCP1700TT, IC3 MCP73831, IC4 MCP1700TT, J1 SWD_PTH_SHROUD, Q1 BSS84, Q2 BSS84, SW1 ROTARTY_ENCODER, U1 NHD-C0216CIZ-FSW, U2 RFM98, U3 RN4020, X1 BU-SMA-V, X2 CRYSTAL-GROUNDED

Commit message: finishing off
Parts:
- removed R11, R12, R14, R15, R2, R3, R6, R7, R8, R9: (no value), resistor:R-EU_R0603
- added RN1, RN2: 330, resistor-dil:4R-NEXB38V
- added RN3: 10k, resistor-dil:4R-NEXB38V
- J1: value SWD_PTH_SHROUD -> SWD_SHROUD_SMD; device dtb:SWD_PTH_SHROUD -> dtb:SWD_SHROUD_SMD
- R13: value (none) -> 22
- R4, R5: value (none) -> 4k7
Connections:
- net AIN1: now also RN3C.2, RN3D.2; no longer R11.2, R14.1
- net GND: now also RN2A.1, RN2B.1, RN2C.1, RN3B.1, RN3C.1; no longer R11.1, R12.1, R3.1, R6.1
- net LED4: now also RN2D.1; no longer R2.1
- net N$10: now also RN2B.2; no longer R6.2
- net N$11: now also RN2D.2; no longer R2.2
- net N$13: now also RN1B.2; no longer R8.2
- net N$14: now also RN1C.2; no longer R9.2
- net N$15: now also RN1A.1; no longer R7.1
- net N$16: now also RN1B.1; no longer R8.1
- net N$17: now also RN1C.1; no longer R9.1
- net N$27: now also RN3A.2, RN3B.2; no longer R12.2, R15.1
- net N$5: now also RN1A.2; no longer R7.2
- net N$6: now also RN2C.2; no longer R3.2
- net VBAT_S: now also RN3A.1; no longer R15.2
- net VBUS: now also RN3D.1; no longer R14.2
Other:
- moved on the sheet: D2, D3, D4, LED5, LED6, LED7

Commit message: adding part values
Parts:
- C1, C13, C15, C3, C4, C9: value (none) -> 1u
- C10, C6: value (none) -> 27p
- C12, C5: value (none) -> 100n
- C2: value (none) -> 4u7
- Q1: value BSS84 -> NX2301
- R1: value (none) -> 10k
- R10, R17: value (none) -> 470
- R16: value (none) -> 4k7
Other:
- note removed: "check can connect both"
- note removed: "connect>"
Changed lines of the file:
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@@
 <part name="GND12" library="supply1" deviceset="GND" device=""/>
 <part name="GND13" library="supply1" deviceset="GND" device=""/>
-<part name="R1" library="resistor" deviceset="R-EU_" device="R0603"/>
+<part name="R1" library="resistor" deviceset="R-EU_" device="R0603" value="10k"/>
 <part name="GND14" library="supply1" deviceset="GND" device=""/>
-<part name="C1" library="resistor" deviceset="C-EU" device="C0603"/>
-<part name="C9" library="resistor" deviceset="C-EU" device="C0603"/>
-<part name="C12" library="resistor" deviceset="C-EU" device="C0603"/>
-<part name="C5" library="resistor" deviceset="C-EU" device="C0603"/>
-<part name="C2" library="resistor" deviceset="C-EU" device="C0603"/>
-<part name="C15" library="resistor" deviceset="C-EU" device="C0603"/>
-<part name="C13" library="resistor" deviceset="C-EU" device="C0603"/>
+<part name="C1" library="resistor" deviceset="C-EU" device="C0603" value="1u"/>
+<part name="C9" library="resistor" deviceset="C-EU" device="C0603" value="1u"/>
+<part name="C12" library="resistor" deviceset="C-EU" device="C0603" value="100n"/>
+<part name="C5" library="resistor" deviceset="C-EU" device="C0603" value="100n"/>
+<part name="C2" library="resistor" deviceset="C-EU" device="C0603" value="4u7"/>
+<part name="C15" library="resistor" deviceset="C-EU" device="C0603" value="1u"/>
+<part name="C13" library="resistor" deviceset="C-EU" device="C0603" value="1u"/>
 <part name="C14" library="resistor" deviceset="C-EU" device="C0603" value="4u7"/>
 <part name="C16" library="resistor" deviceset="C-EU" device="C0603" value="4u7"/>
 <part name="C7" library="resistor" deviceset="C-EU" device="C0603" value="4u7"/>
 <part name="C8" library="resistor" deviceset="C-EU" device="C0603" value="4u7"/>
-<part name="C3" library="resistor" deviceset="C-EU" device="C0603"/>
+<part name="C3" library="resistor" deviceset="C-EU" device="C0603" value="1u"/>
 <part name="C17" library="resistor" deviceset="C-EU" device="C0603" value="4u7"/>
 <part name="GND15" library="supply1" deviceset="GND" device=""/>
@@
 <part name="S3" library="Mine" deviceset="SWITCH-MOMENTARY-2" device="SMD"/>
 <part name="+3V9" library="supply1" deviceset="+3V3" device=""/>
-<part name="Q1" library="transistor-small-signal" deviceset="BSS84" device=""/>
+<part name="Q1" library="transistor-small-signal" deviceset="BSS84" device="" value="NX2301"/>
 <part name="GND30" library="supply1" deviceset="GND" device=""/>
 <part name="+3V8" library="supply1" deviceset="+3V3" device=""/>
-<part name="C4" library="resistor" deviceset="C-EU" device="C0603"/>
+<part name="C4" library="resistor" deviceset="C-EU" device="C0603" value="1u"/>
 <part name="+3V10" library="supply1" deviceset="+3V3" device=""/>
 <part name="R5" library="resistor" deviceset="R-EU_" device="R0603" value="4k7"/>
@@
 <part name="LED6" library="led" deviceset="LED" device="CHIP-LED0805"/>
 <part name="LED1" library="led" deviceset="LED" device="CHIP-LED0805"/>
-<part name="R17" library="resistor" deviceset="R-EU_" device="R0603"/>
+<part name="R17" library="resistor" deviceset="R-EU_" device="R0603" value="470"/>
 <part name="GND31" library="supply1" deviceset="GND" device=""/>
 <part name="GND32" library="supply1" deviceset="GND" device=""/>
 <part name="X2" library="SparkFun-FreqCtrl" deviceset="CRYSTAL-GROUNDED" device=""/>
-<part name="R10" library="resistor" deviceset="R-EU_" device="R0603"/>
-<part name="C10" library="resistor" deviceset="C-EU" device="C0603"/>
-<part name="C6" library="resistor" deviceset="C-EU" device="C0603"/>
+<part name="R10" library="resistor" deviceset="R-EU_" device="R0603" value="470"/>
+<part name="C10" library="resistor" deviceset="C-EU" device="C0603" value="27p"/>
+<part name="C6" library="resistor" deviceset="C-EU" device="C0603" value="27p"/>
 <part name="GND34" library="supply1" deviceset="GND" device=""/>
 <part name="GND35" library="supply1" deviceset="GND" device=""/>
 <part name="GND36" library="supply1" deviceset="GND" device=""/>
-<part name="R16" library="resistor" deviceset="R-EU_" device="R0603"/>
+<part name="R16" library="resistor" deviceset="R-EU_" device="R0603" value="4k7"/>
 <part name="GND37" library="supply1" deviceset="GND" device=""/>
 <part name="L1" library="SparkFun-Passives" deviceset="INDUCTOR" device="0603"/>
@@
 <plain>
 <text x="129.54" y="30.48" size="1.778" layer="91">actually bicolour</text>
-<text x="78.74" y="172.72" size="1.778" layer="91">connect&gt;</text>
-<text x="-25.4" y="165.1" size="1.778" layer="91">connect&gt;</text>
-<text x="-27.94" y="172.72" size="1.778" layer="91">connect&gt;</text>
 <text x="88.9" y="154.94" size="1.778" layer="91">nx2301</text>
 <text x="116.84" y="73.66" size="1.778" layer="91" rot="R180">ESD!</text>
-<text x="-30.48" y="175.26" size="1.778" layer="91">check can connect both </text>
-<text x="71.12" y="175.26" size="1.778" layer="91">check can connect both </text>
 </plain>
 <instances>

Commit message: adding copyright notice
Parts:
- C1, C13, C15, C3, C4, C9: value 1u -> (none)
- C10, C6: value 27p -> (none)
- C12, C5: value 100n -> (none)
- C2: value 4u7 -> (none)
- Q1: value NX2301 -> BSS84
- R1: value 10k -> (none)
- R10, R17: value 470 -> (none)
- R16: value 4k7 -> (none)
Other:
- note added: "Copyright 2014 Matt Brejza"
- note added: "check can connect both"
- note added: "connect>"
Changed lines of the file:
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@@
 <part name="GND12" library="supply1" deviceset="GND" device=""/>
 <part name="GND13" library="supply1" deviceset="GND" device=""/>
-<part name="R1" library="resistor" deviceset="R-EU_" device="R0603" value="10k"/>
+<part name="R1" library="resistor" deviceset="R-EU_" device="R0603"/>
 <part name="GND14" library="supply1" deviceset="GND" device=""/>
-<part name="C1" library="resistor" deviceset="C-EU" device="C0603" value="1u"/>
-<part name="C9" library="resistor" deviceset="C-EU" device="C0603" value="1u"/>
-<part name="C12" library="resistor" deviceset="C-EU" device="C0603" value="100n"/>
-<part name="C5" library="resistor" deviceset="C-EU" device="C0603" value="100n"/>
-<part name="C2" library="resistor" deviceset="C-EU" device="C0603" value="4u7"/>
-<part name="C15" library="resistor" deviceset="C-EU" device="C0603" value="1u"/>
-<part name="C13" library="resistor" deviceset="C-EU" device="C0603" value="1u"/>
+<part name="C1" library="resistor" deviceset="C-EU" device="C0603"/>
+<part name="C9" library="resistor" deviceset="C-EU" device="C0603"/>
+<part name="C12" library="resistor" deviceset="C-EU" device="C0603"/>
+<part name="C5" library="resistor" deviceset="C-EU" device="C0603"/>
+<part name="C2" library="resistor" deviceset="C-EU" device="C0603"/>
+<part name="C15" library="resistor" deviceset="C-EU" device="C0603"/>
+<part name="C13" library="resistor" deviceset="C-EU" device="C0603"/>
 <part name="C14" library="resistor" deviceset="C-EU" device="C0603" value="4u7"/>
 <part name="C16" library="resistor" deviceset="C-EU" device="C0603" value="4u7"/>
 <part name="C7" library="resistor" deviceset="C-EU" device="C0603" value="4u7"/>
 <part name="C8" library="resistor" deviceset="C-EU" device="C0603" value="4u7"/>
-<part name="C3" library="resistor" deviceset="C-EU" device="C0603" value="1u"/>
+<part name="C3" library="resistor" deviceset="C-EU" device="C0603"/>
 <part name="C17" library="resistor" deviceset="C-EU" device="C0603" value="4u7"/>
 <part name="GND15" library="supply1" deviceset="GND" device=""/>
@@
 <part name="S3" library="Mine" deviceset="SWITCH-MOMENTARY-2" device="SMD"/>
 <part name="+3V9" library="supply1" deviceset="+3V3" device=""/>
-<part name="Q1" library="transistor-small-signal" deviceset="BSS84" device="" value="NX2301"/>
+<part name="Q1" library="transistor-small-signal" deviceset="BSS84" device=""/>
 <part name="GND30" library="supply1" deviceset="GND" device=""/>
 <part name="+3V8" library="supply1" deviceset="+3V3" device=""/>
-<part name="C4" library="resistor" deviceset="C-EU" device="C0603" value="1u"/>
+<part name="C4" library="resistor" deviceset="C-EU" device="C0603"/>
 <part name="+3V10" library="supply1" deviceset="+3V3" device=""/>
 <part name="R5" library="resistor" deviceset="R-EU_" device="R0603" value="4k7"/>
@@
 <part name="LED6" library="led" deviceset="LED" device="CHIP-LED0805"/>
 <part name="LED1" library="led" deviceset="LED" device="CHIP-LED0805"/>
-<part name="R17" library="resistor" deviceset="R-EU_" device="R0603" value="470"/>
+<part name="R17" library="resistor" deviceset="R-EU_" device="R0603"/>
 <part name="GND31" library="supply1" deviceset="GND" device=""/>
 <part name="GND32" library="supply1" deviceset="GND" device=""/>
 <part name="X2" library="SparkFun-FreqCtrl" deviceset="CRYSTAL-GROUNDED" device=""/>
-<part name="R10" library="resistor" deviceset="R-EU_" device="R0603" value="470"/>
-<part name="C10" library="resistor" deviceset="C-EU" device="C0603" value="27p"/>
-<part name="C6" library="resistor" deviceset="C-EU" device="C0603" value="27p"/>
+<part name="R10" library="resistor" deviceset="R-EU_" device="R0603"/>
+<part name="C10" library="resistor" deviceset="C-EU" device="C0603"/>
+<part name="C6" library="resistor" deviceset="C-EU" device="C0603"/>
 <part name="GND34" library="supply1" deviceset="GND" device=""/>
 <part name="GND35" library="supply1" deviceset="GND" device=""/>
 <part name="GND36" library="supply1" deviceset="GND" device=""/>
-<part name="R16" library="resistor" deviceset="R-EU_" device="R0603" value="4k7"/>
+<part name="R16" library="resistor" deviceset="R-EU_" device="R0603"/>
 <part name="GND37" library="supply1" deviceset="GND" device=""/>
 <part name="L1" library="SparkFun-Passives" deviceset="INDUCTOR" device="0603"/>
@@
 <plain>
 <text x="129.54" y="30.48" size="1.778" layer="91">actually bicolour</text>
+<text x="78.74" y="172.72" size="1.778" layer="91">connect&gt;</text>
+<text x="-25.4" y="165.1" size="1.778" layer="91">connect&gt;</text>
+<text x="-27.94" y="172.72" size="1.778" layer="91">connect&gt;</text>
 <text x="88.9" y="154.94" size="1.778" layer="91">nx2301</text>
 <text x="116.84" y="73.66" size="1.778" layer="91" rot="R180">ESD!</text>
+<text x="-30.48" y="175.26" size="1.778" layer="91">check can connect both </text>
+<text x="71.12" y="175.26" size="1.778" layer="91">check can connect both </text>
+<text x="-53.34" y="-55.88" size="2.54" layer="97" ratio="15">Copyright 2014 Matt Brejza</text>
+<wire x1="-55.88" y1="-60.96" x2="-55.88" y2="292.1" width="0.4064" layer="97"/>
+<wire x1="-55.88" y1="292.1" x2="190.5" y2="292.1" width="0.4064" layer="97"/>
+<wire x1="190.5" y1="292.1" x2="190.5" y2="-60.96" width="0.4064" layer="97"/>
+<wire x1="190.5" y1="-60.96" x2="-55.88" y2="-60.96" width="0.4064" layer="97"/>
 </plain>
 <instances>

Commit message: minor changes
Other:
- note added: "low leakage"
Changed lines of the file:
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@@
 <wire x1="190.5" y1="292.1" x2="190.5" y2="-60.96" width="0.4064" layer="97"/>
 <wire x1="190.5" y1="-60.96" x2="-55.88" y2="-60.96" width="0.4064" layer="97"/>
+<text x="111.76" y="-20.32" size="1.778" layer="91" rot="R90">low leakage</text>
 </plain>
 <instances>
